File: KiCad/ReAgnus-devboard.kicad_pcb (KiCad board)
At the start: 4 copper layers, 63 x 100 mm, 12 parts, among them J1 Barrel_Jack_Switch, J2 Conn_02x01, J3 Conn_01x01, J4 Conn_01x01, J5 Conn_01x01, J6 Conn_01x01, SW1 SW_SPDT, U1 PLCC-84-Plug, U2 ReAgnus_8375_socket, U3 Agnus_8375_socket

Commit message: Added a microUSB jack for power supply
Parts:
- added J2: USB_B_Micro, Agnus:USB_Micro-B_Unknown_5s_SMT, F.Cu at (160.5, 132.5)
- renumbered J2 to J3, J3 to J4, J4 to J5, J5 to J6, J6 to J7
Routing:
- net /VIN: track 22.1 -> 31.3 mm
Other:
- board text added: "ReAgnus-devboard Rev. 1B"
- board text removed: "ReAgnus-devboard Rev 1A"
